File: FireworksRobot.kicad_pcb (KiCad board)
At the start: 2 copper layers, 66 x 71 mm, 36 parts, among them IC1 SPS440, J1 Conn_01x03, J2 Conthrough, J3 Screw_Terminal_01x02, M1 Motor_DC, M2 Motor_DC, U1 AP2210N-3.3TRG1, U2 STM32F303K8, U3 TB6612FNG, U4 LBR-127HLD, U5 AP2210N-5.0TRG1

Commit message: order
order to elecrow
Parts:
- removed R4: 100, Resistor_SMD:R_0603_1608Metric_Pad1.05x0.95mm_HandSolder
- removed R5: 1k, Resistor_SMD:R_0603_1608Metric_Pad1.05x0.95mm_HandSolder
- removed U4: LBR-127HLD, Connector_PinHeader_2.54mm:PinHeader_1x04_P2.54mm_Vertical
- added J4: Conn_01x05, Connector_PinHeader_2.54mm:PinHeader_1x05_P2.54mm_Vertical, F.Cu at (180.6, 88.9)
- added R6: 1k, Resistor_SMD:R_0603_1608Metric_Pad1.05x0.95mm_HandSolder, F.Cu at (175.0, 99.0)
- added R7: 1k, Resistor_SMD:R_0603_1608Metric_Pad1.05x0.95mm_HandSolder, F.Cu at (175.0, 96.4)
- added R8: 1k, Resistor_SMD:R_0603_1608Metric_Pad1.05x0.95mm_HandSolder, F.Cu at (175.0, 93.6)
- F2: footprint SamacSys_Parts:MF505 -> SamcSys_Parts:MF505
- H1: moved to F.Cu
- IC1: footprint SamacSys_Parts:SPS440 -> SamcSys_Parts:SPS440
- J1: footprint Connector_PinHeader_2.54mm:PinHeader_1x03_P2.54mm_Vertical -> SamcSys_Parts:Conthrough_1x03_P2.54mm_Vertical
- J2: footprint Connector_PinHeader_2.54mm:PinHeader_1x05_P2.54mm_Vertical -> SamcSys_Parts:Conthrough_1x05_P2.54mm_Vertical
- turned H1 to 0 degrees
Connections:
- U2 pad 18: Net-(U2-Pad18) -> /PWMA
- U2 pad 6: Net-(R5-Pad1) -> /COLLECTOR_1
- U2 pad 7: Net-(U2-Pad7) -> /COLLECTOR_2
- U2 pad 9: /PWMA -> /COLLECTOR_3
Routing:
- net /COLLECTOR_2: track 0.00 -> 68.0 mm, vias 0 -> 1
- net /COLLECTOR_1: track 0.00 -> 57.7 mm, vias 0 -> 3
- net Net-(R5-Pad1): track 54.1 -> 0.00 mm, vias 3 -> 0
- net /COLLECTOR_3: track 0.00 -> 50.3 mm, vias 0 -> 1
- net /PWMA: track 4.68 -> 12.5 mm, vias 0 -> 2
- net Net-(R4-Pad1): track 5.57 -> 0.00 mm
- net +3V3: track 92.6 -> 95.3 mm
Other:
- board text added: "3V3"
- board text added: "Designed by TNK."
- board text added: "FireworksRobot Version 1.1"
- board text added: "GND"
- board text added: "NRST"
- board text added: "RX"
- board text added: "SWCLK"
- board text added: "SWDIO"
- board text added: "TX"
- board text added: "https://github.com/ picopicodevil/FireworksRobot.git"

Commit message: Update: シンボル
Parts:
- removed the D4 at (154.0, 135.0)
- removed the D5 at (146.0, 135.0)
- removed D6, D7: WS2812B, LED_SMD:LED_WS2812B_PLCC4_5.0x5.0mm_P3.2mm
- added D1: LED_RABG, LED_THT:LED_D5.0mm-4_RGB, F.Cu at (144.8, 140.4)
- added D3: LED_RABG, LED_THT:LED_D5.0mm-4_RGB, F.Cu at (151.4, 140.4)
- added R1: 62, Resistor_SMD:R_0603_1608Metric_Pad1.05x0.95mm_HandSolder, F.Cu at (145.0, 134.0)
- added R2: 62, Resistor_SMD:R_0603_1608Metric_Pad1.05x0.95mm_HandSolder, F.Cu at (147.9, 134.0)
- added R3: 200, Resistor_SMD:R_0603_1608Metric_Pad1.05x0.95mm_HandSolder, F.Cu at (142.1, 134.0)
- added R6: 62, Resistor_SMD:R_0603_1608Metric_Pad1.05x0.95mm_HandSolder, F.Cu at (155.1, 134.0)
- added R7: 62, Resistor_SMD:R_0603_1608Metric_Pad1.05x0.95mm_HandSolder, F.Cu at (158.0, 134.0)
- added R8: 200, Resistor_SMD:R_0603_1608Metric_Pad1.05x0.95mm_HandSolder, F.Cu at (152.2, 134.0)
- F2: footprint SamcSys_Parts:MF505 -> SamacSys_Parts:MF505
- IC1: footprint SamcSys_Parts:SPS440 -> SamacSys_Parts:SPS440
- J1: footprint SamcSys_Parts:Conthrough_1x03_P2.54mm_Vertical -> SamacSys_Parts:Conthrough_1x03_P2.54mm_Vertical
- J2: footprint SamcSys_Parts:Conthrough_1x05_P2.54mm_Vertical -> SamacSys_Parts:Conthrough_1x05_P2.54mm_Vertical
- renumbered C2 to C1, C3 to C2, C6 to C3, C7 to C4, C1 to C5, C4 to C6, C5 to C7, D1 to D2, D2 to D4, D3 to D5, R6 to R10, R7 to R11, R8 to R12, R2 to R4, R3 to R5, R1 to R9, U5 to U2, U2 to U3, U3 to U4
Connections:
- U3 pad 26: Net-(U2-Pad26) -> LED_G
- U3 pad 27: Net-(U2-Pad27) -> LED_B
- U3 pad 28: Net-(D4-Pad4) -> LED_R
Routing:
- net LED_R: track 0.00 -> 58.1 mm, vias 0 -> 3
- net +5V: track 70.8 -> 12.9 mm, vias 2 -> 0
- net LED_B: track 0.00 -> 56.5 mm, vias 0 -> 3
- net LED_G: track 0.00 -> 55.3 mm, vias 0 -> 3
- net Net-(D4-Pad4): track 46.7 -> 0.00 mm, vias 2 -> 0
- net +3V3: track 95.3 -> 140.2 mm, vias 3 -> 4
- net Net-(D5-Pad2) (its old number): track 6.89 -> 0.00 mm
- net Net-(D3-Pad4): track 0.00 -> 6.68 mm
- net Net-(D1-Pad1): track 0.00 -> 6.64 mm
- net /COLLECTOR_2: track 68.0 -> 74.6 mm
- net Net-(D1-Pad3): track 0.00 -> 6.49 mm
- net Net-(D3-Pad3): track 0.00 -> 6.01 mm
- net Net-(D3-Pad1): track 0.00 -> 5.86 mm
- net Net-(D1-Pad4): track 0.00 -> 5.82 mm
- net Net-(D6-Pad2): track 4.48 -> 0.00 mm
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