File: FireworksRobot.sch (KiCad schematic (older format))
At the start: 36 parts, among them IC1 SPS440, J1 Conn_01x03, J2 Conthrough, J3 Screw_Terminal_01x02, M1 Motor_DC, M2 Motor_DC, U1 AP2210N-3.3TRG1, U2 STM32F303K8, U3 TB6612FNG, U4 LBR-127HLD, U5 AP2210N-5.0TRG1

Commit message: order
order to elecrow
Parts:
- removed R4: 100, Resistor_SMD:R_0603_1608Metric_Pad1.05x0.95mm_HandSolder, symbol Device:R
- removed R5: 1k, Resistor_SMD:R_0603_1608Metric_Pad1.05x0.95mm_HandSolder, symbol Device:R
- removed U4: LBR-127HLD, Connector_PinHeader_2.54mm:PinHeader_1x04_P2.54mm_Vertical, symbol SamacSys_Parts:LBR-127HLD
- added J4: Conn_01x05, Connector_PinHeader_2.54mm:PinHeader_1x05_P2.54mm_Vertical, symbol Connector_Generic:Conn_01x05
- added R6, R7, R8: 1k, Resistor_SMD:R_0603_1608Metric_Pad1.05x0.95mm_HandSolder, symbol Device:R
- F2: footprint SamacSys_Parts:MF505 -> SamcSys_Parts:MF505
- IC1: footprint SamacSys_Parts:SPS440 -> SamcSys_Parts:SPS440
- J1: footprint Connector_PinHeader_2.54mm:PinHeader_1x03_P2.54mm_Vertical -> SamcSys_Parts:Conthrough_1x03_P2.54mm_Vertical
- J2: footprint Connector_PinHeader_2.54mm:PinHeader_1x05_P2.54mm_Vertical -> SamcSys_Parts:Conthrough_1x05_P2.54mm_Vertical
Connections:
- net +3V3: now also J4.2 (Pin_2), R6.2, R7.2, R8.2
- net GND: now also J4.1 (Pin_1)
- net PWMA: now also U2.18 (PA8); no longer U2.9 (PA3)
- net COLLECTOR_1: now reaches U2.6 (PA0)
- net COLLECTOR_1: now also J4.3 (Pin_3), R8.1
- net COLLECTOR_2: now reaches U2.7 (PA1)
- net COLLECTOR_2: now also J4.4 (Pin_4), R7.1
- new net COLLECTOR_3: J4.5 (Pin_5), R6.1, U2.9 (PA3)
- no-connect marks 10 -> 8
Other:
- moved on the sheet: H1, H2, H3, H4

Commit message: Update: シンボル
Parts:
- removed D4, D5, D6, D7: WS2812B, LED_SMD:LED_WS2812B_PLCC4_5.0x5.0mm_P3.2mm, symbol LED:WS2812B
- added D1, D3: LED_RABG, LED_THT:LED_D5.0mm-4_RGB, symbol Device:LED_RABG
- added R1, R2, R6, R7: 62, Resistor_SMD:R_0603_1608Metric_Pad1.05x0.95mm_HandSolder, symbol Device:R
- added R3, R8: 200, Resistor_SMD:R_0603_1608Metric_Pad1.05x0.95mm_HandSolder, symbol Device:R
- F2: footprint SamcSys_Parts:MF505 -> SamacSys_Parts:MF505
- IC1: footprint SamcSys_Parts:SPS440 -> SamacSys_Parts:SPS440
- J1: footprint SamcSys_Parts:Conthrough_1x03_P2.54mm_Vertical -> SamacSys_Parts:Conthrough_1x03_P2.54mm_Vertical
- J2: footprint SamcSys_Parts:Conthrough_1x05_P2.54mm_Vertical -> SamacSys_Parts:Conthrough_1x05_P2.54mm_Vertical
- renumbered C2 to C1, C3 to C2, C6 to C3, C7 to C4, C1 to C5, C4 to C6, C5 to C7, D1 to D2, D2 to D4, D3 to D5, R6 to R10, R7 to R11, R8 to R12, R2 to R4, R3 to R5, R1 to R9, U5 to U2, U2 to U3, U3 to U4
Connections:
- net +3V3: now also D1.2 (A), D3.2 (A)
- net LED_G: now reaches U3.26 (PB3)
- net LED_G: now also R2.2, R7.2
- net LED_B: now reaches U3.27 (PB4)
- net LED_B: now also R1.2, R6.2
- net LED_R: now reaches U3.28 (PB5)
- net LED_R: now also R3.2, R8.2
- new net: D3.1 (RK), R8.1
- new net: D3.3 (BK), R6.1
- new net: D3.4 (GK), R7.1
- new net: D1.1 (RK), R3.1
- new net: D1.3 (BK), R1.1
- new net: D1.4 (GK), R2.1
- no-connect marks 8 -> 5
